Commit message: 修复差速轮转向：翻转两驱动轮关节axis为0 0 -1，前进指令对应前进运动

File: src/robot_description/urdf/robot.xacro (robot description, xacro)
@@ -49,5 +49,5 @@
     <child link="left_wheel_link"/>
     <origin xyz="0.15 0.175 0.075" rpy="${pi/2} 0 0"/>
-    <axis xyz="0 0 1"/>
+    <axis xyz="0 0 -1"/>
   </joint>
   <link name="left_wheel_link">
@@ -81,5 +81,5 @@
     <child link="right_wheel_link"/>
     <origin xyz="0.15 -0.175 0.075" rpy="${pi/2} 0 0"/>
-    <axis xyz="0 0 1"/>
+    <axis xyz="0 0 -1"/>
   </joint>
   <link name="right_wheel_link">
