Commit message: 同步VM调试状态：改进URDF惯性/碰撞、精简nav2参数、更新地图与RViz配置

File: src/robot_description/urdf/gazebo.xacro (robot description, xacro)
@@ -1,34 +1,20 @@
 <?xml version="1.0"?>
 <robot xmlns:xacro="http://www.ros.org/wiki/xacro" name="gazebo_plugins">
-  <!-- ============================================================ -->
-  <!-- Gazebo 差速驱动插件                                           -->
-  <!-- 使用 gazebo_ros_diff_drive 实现差速驱动控制                    -->
-  <!-- 发布话题: /cmd_vel, /odom, /tf                               -->
-  <!-- ============================================================ -->
+  <!-- 差速驱动插件 -->
   <gazebo>
     <plugin name="diff_drive" filename="libgazebo_ros_diff_drive.so">
-      <!-- 发布和订阅的话题 -->
-      <ros>
-        <namespace>/</namespace>
-      </ros>
-      <!-- 更新频率 (Hz) -->
+      <ros><namespace>/</namespace></ros>
       <update_rate>50</update_rate>
-      <!-- 轮子关节名称 -->
       <left_joint>left_wheel_joint</left_joint>
       <right_joint>right_wheel_joint</right_joint>
-      <!-- 轮子参数 -->
-      <wheel_separation>0.35</wheel_separation>   <!-- 2 * 0.175 = 0.35m -->
+      <wheel_separation>0.35</wheel_separation>
       <wheel_diameter>0.15</wheel_diameter>
-      <!-- 速度限制 (与需求文档一致) -->
-      <max_wheel_torque>20.0</max_wheel_torque>
-      <max_wheel_acceleration>2.0</max_wheel_acceleration>
-      <!-- 发布里程计 -->
+      <max_wheel_torque>50.0</max_wheel_torque>
+      <max_wheel_acceleration>10.0</max_wheel_acceleration>
       <publish_odom>true</publish_odom>
       <publish_odom_tf>true</publish_odom_tf>
       <publish_wheel_tf>true</publish_wheel_tf>
-      <!-- 坐标系 -->
       <odometry_frame>odom</odometry_frame>
       <robot_base_frame>base_link</robot_base_frame>
-      <!-- 协方差矩阵 (3x3行主序) -->
       <covariance_x>0.0001</covariance_x>
       <covariance_y>0.0001</covariance_y>
@@ -36,22 +22,17 @@
     </plugin>
   </gazebo>
-  <!-- ============================================================ -->
-  <!-- Gazebo 激光雷达插件                                           -->
-  <!-- 使用 gazebo_ros_laser 发布 LaserScan 消息                     -->
-  <!-- 话题: /scan, 坐标系: laser_link                               -->
-  <!-- ============================================================ -->
+  <!-- 2D激光雷达 - 单线360度水平扫描 -->
   <gazebo reference="laser_link">
     <sensor type="ray" name="laser_sensor">
       <always_on>true</always_on>
-      <update_rate>10</update_rate>   <!-- 10Hz 扫描频率 -->
+      <update_rate>10</update_rate>
       <visualize>true</visualize>
-      <pose>0 0 0 0 0 0</pose>
       <ray>
         <scan>
           <horizontal>
-            <samples>360</samples>        <!-- 360度扫描 -->
+            <samples>360</samples>
             <resolution>1</resolution>
             <min_angle>0</min_angle>
-            <max_angle>6.283185307179586</max_angle>   <!-- 2*pi -->
+            <max_angle>6.283185307179586</max_angle>
           </horizontal>
           <vertical>
@@ -63,6 +44,6 @@
         </scan>
         <range>
-          <min>0.1</min>                  <!-- 最小扫描距离 0.1m -->
-          <max>5.0</max>                  <!-- 最大扫描距离 5.0m -->
+          <min>0.1</min>
+          <max>5.0</max>
           <resolution>0.01</resolution>
         </range>
@@ -74,4 +55,5 @@
       </ray>
       <plugin name="laser_plugin" filename="libgazebo_ros_ray_sensor.so">
+        <ros><namespace>/</namespace></ros>
         <frame_name>laser_link</frame_name>
         <output_type>sensor_msgs/LaserScan</output_type>
@@ -80,31 +62,21 @@
     </sensor>
   </gazebo>
-  <!-- ============================================================ -->
-  <!-- Gazebo 视觉材质配置                                           -->
-  <!-- ============================================================ -->
-  <!-- base_link 蓝色金属质感 -->
+  <!-- 材质 -->
   <gazebo reference="base_link">
     <material>Gazebo/Blue</material>
-    <mu1>0.8</mu1>
-    <mu2>0.8</mu2>
+    <mu1>0.8</mu1><mu2>0.8</mu2>
   </gazebo>
-  <!-- 驱动轮 深灰色橡胶质感 -->
   <gazebo reference="left_wheel_link">
     <material>Gazebo/DarkGrey</material>
-    <mu1>1.5</mu1>
-    <mu2>1.5</mu2>
+    <mu1>1.5</mu1><mu2>1.5</mu2>
   </gazebo>
   <gazebo reference="right_wheel_link">
     <material>Gazebo/DarkGrey</material>
-    <mu1>1.0</mu1>
-    <mu2>1.0</mu2>
+    <mu1>1.5</mu1><mu2>1.5</mu2>
   </gazebo>
-  <!-- 随动轮 -->
   <gazebo reference="caster_wheel_link">
     <material>Gazebo/DarkGrey</material>
-    <mu1>1.5</mu1>
-    <mu2>1.5</mu2>
+    <mu1>0.1</mu1><mu2>0.1</mu2>
   </gazebo>
-  <!-- 激光雷达 -->
   <gazebo reference="laser_link">
     <material>Gazebo/Black</material>

File: src/robot_description/urdf/robot.xacro (robot description, xacro)
@@ -1,79 +1,176 @@
 <?xml version="1.0"?>
 <robot xmlns:xacro="http://www.ros.org/wiki/xacro" name="articubot_robot">
+  <!-- ============================================================ -->
+  <!-- 包含材质定义                                                    -->
+  <!-- ============================================================ -->
   <xacro:include filename="$(find robot_description)/urdf/materials.xacro"/>
-  <xacro:property name="M_total" value="2.0"/>
-  <xacro:property name="M_wheel" value="0.2"/>
-  <xacro:property name="M_caster" value="0.1"/>
-  <xacro:property name="M_body" value="${M_total - 2*M_wheel - M_caster}"/>
-  <!-- base_link: 0.5x0.3x0.25m, 蓝色 -->
+  <!-- ============================================================ -->
+  <!-- 全局参数                                                       -->
+  <!-- ============================================================ -->
+  <xacro:property name="M_total" value="2.0"/>        <!-- 总质量 (kg) -->
+  <xacro:property name="M_wheel" value="0.2"/>        <!-- 驱动轮质量 (kg) -->
+  <xacro:property name="M_caster" value="0.1"/>       <!-- 随动轮质量 (kg) -->
+  <xacro:property name="M_body" value="${M_total - 2*M_wheel - M_caster}"/> <!-- 主体质量 (kg) -->
+  <!-- ============================================================ -->
+  <!-- 主体 (base_link)                                              -->
+  <!-- 尺寸: 0.5m x 0.3m x 0.25m                                    -->
+  <!-- ============================================================ -->
   <link name="base_link">
     <visual>
       <origin xyz="0 0 ${0.25/2}" rpy="0 0 0"/>
-      <geometry><box size="0.5 0.3 0.25"/></geometry>
+      <geometry>
+        <box size="0.5 0.3 0.25"/>
+      </geometry>
       <material name="robot_blue"/>
     </visual>
     <collision>
       <origin xyz="0 0 ${0.25/2}" rpy="0 0 0"/>
-      <geometry><box size="0.48 0.28 0.25"/></geometry>
+      <geometry>
+        <box size="0.5 0.3 0.25"/>
+      </geometry>
     </collision>
     <inertial>
       <origin xyz="0 0 ${0.25/2}" rpy="0 0 0"/>
       <mass value="${M_body}"/>
-      <inertia ixx="${M_body*(0.3*0.3+0.25*0.25)/12}" ixy="0.0" ixz="0.0"
-               iyy="${M_body*(0.5*0.5+0.25*0.25)/12}" iyz="0.0"
+      <inertia ixx="${M_body*(0.3*0.3+0.25*0.25)/12}"
+               ixy="0.0"
+               ixz="0.0"
+               iyy="${M_body*(0.5*0.5+0.25*0.25)/12}"
+               iyz="0.0"
                izz="${M_body*(0.5*0.5+0.3*0.3)/12}"/>
     </inertial>
   </link>
-  <!-- 左驱动轮 -->
+  <!-- ============================================================ -->
+  <!-- 左驱动轮 (left_wheel_link)                                    -->
+  <!-- 直径: 0.15m, 宽度: 0.05m, 中心: (0.15, 0.175, 0.075)        -->
+  <!-- ============================================================ -->
   <joint name="left_wheel_joint" type="continuous">
-    <parent link="base_link"/><child link="left_wheel_link"/>
+    <parent link="base_link"/>
+    <child link="left_wheel_link"/>
     <origin xyz="0.15 0.175 0.075" rpy="${pi/2} 0 0"/>
     <axis xyz="0 0 1"/>
   </joint>
   <link name="left_wheel_link">
-    <visual><geometry><cylinder radius="0.075" length="0.05"/></geometry><material name="wheel_dark_grey"/></visual>
-    <collision><geometry><cylinder radius="0.075" length="0.05"/></geometry></collision>
+    <visual>
+      <geometry>
+        <cylinder radius="${0.15/2}" length="0.05"/>
+      </geometry>
+      <material name="wheel_dark_grey"/>
+    </visual>
+    <collision>
+      <geometry>
+        <cylinder radius="${0.15/2}" length="0.05"/>
+      </geometry>
+    </collision>
     <inertial>
       <mass value="${M_wheel}"/>
-      <inertia ixx="${M_wheel*0.075*0.075/2}" ixy="0" ixz="0" iyy="${M_wheel*0.075*0.075/2}" iyz="0" izz="${M_wheel*0.075*0.075/2}"/>
+      <inertia ixx="${M_wheel*(3*(0.15/2)*(0.15/2)+0.05*0.05)/12}"
+               ixy="0.0"
+               ixz="0.0"
+               iyy="${M_wheel*(3*(0.15/2)*(0.15/2)+0.05*0.05)/12}"
+               iyz="0.0"
+               izz="${M_wheel*(0.15/2)*(0.15/2)/2}"/>
     </inertial>
   </link>
-  <!-- 右驱动轮 -->
+  <!-- ============================================================ -->
+  <!-- 右驱动轮 (right_wheel_link)                                   -->
+  <!-- 直径: 0.15m, 宽度: 0.05m, 中心: (0.15, -0.175, 0.075)       -->
+  <!-- ============================================================ -->
   <joint name="right_wheel_joint" type="continuous">
-    <parent link="base_link"/><child link="right_wheel_link"/>
+    <parent link="base_link"/>
+    <child link="right_wheel_link"/>
     <origin xyz="0.15 -0.175 0.075" rpy="${pi/2} 0 0"/>
     <axis xyz="0 0 1"/>
   </joint>
   <link name="right_wheel_link">
-    <visual><geometry><cylinder radius="0.075" length="0.05"/></geometry><material name="wheel_dark_grey"/></visual>
-    <collision><geometry><cylinder radius="0.075" length="0.05"/></geometry></collision>
+    <visual>
+      <geometry>
+        <cylinder radius="${0.15/2}" length="0.05"/>
+      </geometry>
+      <material name="wheel_dark_grey"/>
+    </visual>
+    <collision>
+      <geometry>
+        <cylinder radius="${0.15/2}" length="0.05"/>
+      </geometry>
+    </collision>
     <inertial>
       <mass value="${M_wheel}"/>
-      <inertia ixx="${M_wheel*0.075*0.075/2}" ixy="0" ixz="0" iyy="${M_wheel*0.075*0.075/2}" iyz="0" izz="${M_wheel*0.075*0.075/2}"/>
+      <inertia ixx="${M_wheel*(3*(0.15/2)*(0.15/2)+0.05*0.05)/12}"
+               ixy="0.0"
+               ixz="0.0"
+               iyy="${M_wheel*(3*(0.15/2)*(0.15/2)+0.05*0.05)/12}"
+               iyz="0.0"
+               izz="${M_wheel*(0.15/2)*(0.15/2)/2}"/>
     </inertial>
   </link>
-  <!-- 随动轮 (固定关节，不旋转) -->
+  <!-- ============================================================ -->
+  <!-- 随动轮 (caster_wheel_link)                                    -->
+  <!-- 直径: 0.10m, 宽度: 0.05m, 中心: (-0.15, 0, 0.05)            -->
+  <!-- 固定关节 (fixed joint)                                        -->
+  <!-- ============================================================ -->
   <joint name="caster_wheel_joint" type="fixed">
-    <parent link="base_link"/><child link="caster_wheel_link"/>
+    <parent link="base_link"/>
+    <child link="caster_wheel_link"/>
     <origin xyz="-0.15 0.0 0.05" rpy="${pi/2} 0 0"/>
   </joint>
   <link name="caster_wheel_link">
-    <visual><geometry><cylinder radius="0.05" length="0.05"/></geometry><material name="caster_grey"/></visual>
-    <collision><geometry><cylinder radius="0.05" length="0.05"/></geometry></collision>
+    <visual>
+      <geometry>
+        <cylinder radius="${0.10/2}" length="0.05"/>
+      </geometry>
+      <material name="caster_grey"/>
+    </visual>
+    <collision>
+      <geometry>
+        <cylinder radius="${0.10/2}" length="0.05"/>
+      </geometry>
+    </collision>
     <inertial>
       <mass value="${M_caster}"/>
-      <inertia ixx="${M_caster*0.05*0.05/2}" ixy="0" ixz="0" iyy="${M_caster*0.05*0.05/2}" iyz="0" izz="${M_caster*0.05*0.05/2}"/>
+      <inertia ixx="${M_caster*(3*(0.10/2)*(0.10/2)+0.05*0.05)/12}"
+               ixy="0.0"
+               ixz="0.0"
+               iyy="${M_caster*(3*(0.10/2)*(0.10/2)+0.05*0.05)/12}"
+               iyz="0.0"
+               izz="${M_caster*(0.10/2)*(0.10/2)/2}"/>
     </inertial>
   </link>
-  <!-- 激光雷达 z=0.27m, fixed joint -->
+  <!-- ============================================================ -->
+  <!-- 激光雷达 (laser_link)                                         -->
+  <!-- 安装在主体顶部中心: (0, 0, 0.25)                               -->
+  <!-- ============================================================ -->
   <joint name="laser_joint" type="fixed">
-    <parent link="base_link"/><child link="laser_link"/>
-    <origin xyz="0.0 0.0 0.27" rpy="0 0 0"/>
+    <parent link="base_link"/>
+    <child link="laser_link"/>
+    <origin xyz="0.0 0.0 0.26" rpy="0 0 0"/>
   </joint>
   <link name="laser_link">
-    <visual><geometry><cylinder radius="0.04" length="0.03"/></geometry><material name="lidar_dark"/></visual>
-    <collision><geometry><cylinder radius="0.04" length="0.03"/></geometry></collision>
-    <inertial><mass value="0.01"/><inertia ixx="0.000001" ixy="0" ixz="0" iyy="0.000001" iyz="0" izz="0.000001"/></inertial>
+    <visual>
+      <origin xyz="0 0 0" rpy="0 0 0"/>
+      <geometry>
+        <cylinder radius="0.04" length="0.03"/>
+      </geometry>
+      <material name="lidar_dark"/>
+    </visual>
+    <collision>
+      <origin xyz="0 0 0" rpy="0 0 0"/>
+      <geometry>
+        <cylinder radius="0.04" length="0.03"/>
+      </geometry>
+    </collision>
+    <inertial>
+      <mass value="0.01"/>
+      <inertia ixx="0.000001"
+               ixy="0.0"
+               ixz="0.0"
+               iyy="0.000001"
+               iyz="0.0"
+               izz="0.000001"/>
+    </inertial>
   </link>
+  <!-- ============================================================ -->
+  <!-- Gazebo 插件配置                                               -->
+  <!-- ============================================================ -->
   <xacro:include filename="$(find robot_description)/urdf/gazebo.xacro"/>
 </robot>

Commit message: 修复转向不灵敏：随动轮碰撞体改为无摩擦球面，消除旋转拖拽

File: src/robot_description/urdf/gazebo.xacro (robot description, xacro)
@@ -80,5 +80,6 @@
   <gazebo reference="caster_wheel_link">
     <material>Gazebo/DarkGrey</material>
-    <mu1>0.1</mu1><mu2>0.1</mu2>
+    <!-- 随动轮球面碰撞体设为无摩擦, 让小车旋转时不被随动轮拖拽 -->
+    <mu1>0.0</mu1><mu2>0.0</mu2>
   </gazebo>
   <gazebo reference="laser_link">

File: src/robot_description/urdf/robot.xacro (robot description, xacro)
@@ -122,7 +122,8 @@
       <material name="caster_grey"/>
     </visual>
+    <!-- 碰撞体用球面: 随动轮无法转向, 球面可在各方向自由滑动, 避免阻碍小车旋转 -->
     <collision>
       <geometry>
-        <cylinder radius="${0.10/2}" length="0.05"/>
+        <sphere radius="${0.10/2}"/>
       </geometry>
     </collision>

Commit message: 修复转向不灵敏根因：车身碰撞体抬高离地0.05m消除底盘拖地；恢复扭矩50；nav2 scan话题与代价地图观测源修正；新增导航验证脚本

File: src/robot_description/urdf/gazebo.xacro (robot description, xacro)
@@ -10,6 +10,6 @@
       <wheel_separation>0.35</wheel_separation>
       <wheel_diameter>0.15</wheel_diameter>
-      <max_wheel_torque>200.0</max_wheel_torque>
-      <max_wheel_acceleration>100.0</max_wheel_acceleration>
+      <max_wheel_torque>50.0</max_wheel_torque>
+      <max_wheel_acceleration>10.0</max_wheel_acceleration>
       <publish_odom>true</publish_odom>
       <publish_odom_tf>true</publish_odom_tf>

File: src/robot_description/urdf/robot.xacro (robot description, xacro)
@@ -24,8 +24,9 @@
       <material name="robot_blue"/>
     </visual>
+    <!-- 碰撞体抬高0.05m离地, 避免车身底盘拖地(否则严重阻碍旋转); 视觉体仍为规范0.25高 -->
     <collision>
-      <origin xyz="0 0 ${0.25/2}" rpy="0 0 0"/>
+      <origin xyz="0 0 0.15" rpy="0 0 0"/>
       <geometry>
-        <box size="0.5 0.3 0.25"/>
+        <box size="0.5 0.3 0.20"/>
       </geometry>
     </collision>
